File: uino-328th.brd (EAGLE design)
At the start: 68.6 x 53.3 mm, 38 parts, among them J1 CON_TERMINAL_BLOCK_02-5MM, J2 USB_MICRO_B_2.0-TH, U1 V_REG_MCP170X, U2 PIC16F1454-P, U3 ATMEGA328P-P

Commit message: Some minor final changes.
Connections:
- removed net N$6: J2.4
Routing:
- net GND: track 0.00 -> 7.89 mm, vias 19 -> 29
- net N$4: track 14.6 -> 16.4 mm
- net N$3: track 16.8 -> 18.7 mm
Changed lines of the file:
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@@
 <setting verticaltext="up"/>
 </settings>
-<grid distance="0.05" unitdist="inch" unit="mil" style="lines" multiple="1" display="yes" altdistance="12.5" altunitdist="mil" altunit="mil"/>
+<grid distance="0.05" unitdist="inch" unit="mm" style="lines" multiple="1" display="yes" altdistance="12.5" altunitdist="mil" altunit="mil"/>
 <layers>
 <layer number="1" name="Top" color="4" fill="1" visible="yes" active="yes"/>
@@
 <attribute name="VALUE" x="60.452" y="31.75" size="1.27" layer="27" rot="R270"/>
 </element>
-<element name="J2" library="adi-misc" package="ZX62D-AB-5P8" value="USB_MICRO_B_2.0-TH" x="1.905" y="38.1" rot="R270"/>
 <element name="U3" library="adi-atmega" package="DIL28-3" value="ATMEGA328P-P" x="46.99" y="16.51" smashed="yes" rot="R180">
 <attribute name="NAME" x="65.0875" y="16.51" size="1.016" layer="25" ratio="18"/>
@@
 <attribute name="VALUE" x="9.2075" y="53.975" size="0.8128" layer="27" ratio="10" rot="R180"/>
 </element>
+<element name="J2" library="adi-misc" package="ZX62D-AB-5P8" value="USB_MICRO_B_2.0-TH" x="1.905" y="38.1" rot="R270"/>
 </elements>
 <signals>
@@
 <wire x1="20.955" y1="8.89" x2="20.955" y2="7.62" width="0.8128" layer="1"/>
 </signal>
-<signal name="GND" airwireshidden="yes">
+<signal name="GND">
 <contactref element="JP4" pad="4"/>
 <contactref element="JP4" pad="5"/>
@@
 <contactref element="C2" pad="1"/>
 <contactref element="U2" pad="14"/>
-<contactref element="J2" pad="S1"/>
-<contactref element="J2" pad="5"/>
-<contactref element="J2" pad="S2"/>
 <contactref element="J3" pad="3"/>
 <contactref element="D6" pad="K"/>
@@
 <via x="18.415" y="33.02" extent="1-16" drill="0.400659375"/>
 <via x="43.815" y="51.7525" extent="1-16" drill="0.400659375"/>
-<wire x1="1.905" y1="33.925" x2="4.605" y2="36.8" width="0" layer="19" extent="1-1"/>
+<contactref element="J2" pad="S1"/>
+<contactref element="J2" pad="S2"/>
+<contactref element="J2" pad="5"/>
+<wire x1="4.605" y1="36.8" x2="7.2725" y2="36.8" width="0.254" layer="1"/>
+<wire x1="7.2725" y1="36.8" x2="9.8425" y2="39.37" width="0.254" layer="1"/>
+<wire x1="9.8425" y1="39.37" x2="11.43" y2="39.37" width="0.254" layer="1"/>
+<via x="41.91" y="17.4625" extent="1-16" drill="0.400659375"/>
+<via x="49.53" y="25.7175" extent="1-16" drill="0.400659375"/>
+<via x="59.69" y="26.67" extent="1-16" drill="0.400659375"/>
+<via x="62.23" y="48.5775" extent="1-16" drill="0.400659375"/>
+<via x="59.69" y="48.5775" extent="1-16" drill="0.400659375"/>
+<via x="54.61" y="49.53" extent="1-16" drill="0.400659375"/>
+<via x="57.15" y="48.895" extent="1-16" drill="0.400659375"/>
+<via x="52.07" y="49.53" extent="1-16" drill="0.400659375"/>
+<via x="37.7825" y="49.53" extent="1-16" drill="0.400659375"/>
+<via x="21.2725" y="38.4175" extent="1-16" drill="0.400659375"/>
 </signal>
 <signal name="A0">
@@
 <wire x1="54.2925" y1="31.115" x2="54.2925" y2="42.2275" width="0.4064" layer="1"/>
 <wire x1="54.2925" y1="42.2275" x2="45.72" y2="50.8" width="0.4064" layer="1"/>
-</signal>
-<signal name="N$3">
-<contactref element="J2" pad="2"/>
-<contactref element="U2" pad="12"/>
-<wire x1="4.605" y1="38.75" x2="6.6825" y2="38.75" width="0.254" layer="1"/>
-<via x="8.89" y="40.9575" extent="1-16" drill="0.400659375"/>
-<wire x1="8.89" y1="40.9575" x2="17.78" y2="40.9575" width="0.4064" layer="16"/>
-<wire x1="17.78" y1="40.9575" x2="19.05" y2="42.2275" width="0.4064" layer="16"/>
-<wire x1="19.05" y1="42.2275" x2="19.05" y2="43.18" width="0.4064" layer="16"/>
-<wire x1="6.6825" y1="38.75" x2="8.89" y2="40.9575" width="0.254" layer="1"/>
-</signal>
-<signal name="N$4">
-<contactref element="J2" pad="3"/>
-<contactref element="U2" pad="13"/>
-<wire x1="4.605" y1="38.1" x2="6.985" y2="38.1" width="0.254" layer="1"/>
-<wire x1="6.985" y1="38.1" x2="8.5725" y2="39.6875" width="0.254" layer="1"/>
-<wire x1="8.5725" y1="39.6875" x2="9.2075" y2="39.6875" width="0.4064" layer="1"/>
-<wire x1="9.2075" y1="39.6875" x2="10.4775" y2="40.9575" width="0.4064" layer="1"/>
-<wire x1="10.4775" y1="40.9575" x2="15.24" y2="40.9575" width="0.4064" layer="1"/>
-<wire x1="15.24" y1="40.9575" x2="16.51" y2="42.2275" width="0.4064" layer="1"/>
-<wire x1="16.51" y1="42.2275" x2="16.51" y2="43.18" width="0.4064" layer="1"/>
-</signal>
-<signal name="N$6">
-<contactref element="J2" pad="4"/>
 </signal>
 <signal name="CLKIN">
@@
 </signal>
 <signal name="VBUS">
-<contactref element="J2" pad="1"/>
 <contactref element="F1" pad="P$1"/>
-<wire x1="4.605" y1="39.4" x2="6.38" y2="39.4" width="0.254" layer="1"/>
 <wire x1="6.38" y1="39.4" x2="7.3025" y2="40.3225" width="0.254" layer="1"/>
 <wire x1="7.3025" y1="40.3225" x2="7.3025" y2="40.9575" width="0.4064" layer="1"/>
@@
 <wire x1="19.3675" y1="29.845" x2="24.765" y2="29.845" width="0.6096" layer="16"/>
 <wire x1="24.765" y1="29.845" x2="25.4" y2="30.48" width="0.6096" layer="16"/>
+<contactref element="J2" pad="1"/>
+<wire x1="4.605" y1="39.4" x2="6.38" y2="39.4" width="0.254" layer="1"/>
 </signal>
 <signal name="N$14">
@@
 <wire x1="26.67" y1="22.86" x2="26.67" y2="7.62" width="0.6096" layer="1"/>
 </signal>
+<signal name="N$3">
+<contactref element="J2" pad="2"/>
+<contactref element="U2" pad="12"/>
+<wire x1="4.605" y1="38.75" x2="6.6825" y2="38.75" width="0.254" layer="1"/>
+<wire x1="6.6825" y1="38.75" x2="8.89" y2="40.9575" width="0.254" layer="1"/>
+<via x="8.89" y="40.9575" extent="1-16" drill="0.400659375"/>
+<wire x1="8.89" y1="40.9575" x2="9.525" y2="41.5925" width="0.4064" layer="16"/>
+<wire x1="9.525" y1="41.5925" x2="12.3825" y2="41.5925" width="0.4064" layer="16"/>
+<wire x1="12.3825" y1="41.5925" x2="13.97" y2="40.005" width="0.4064" layer="16"/>
+<wire x1="13.97" y1="40.005" x2="17.78" y2="40.005" width="0.4064" layer="16"/>
+<wire x1="17.78" y1="40.005" x2="19.05" y2="41.275" width="0.4064" layer="16"/>
+<wire x1="19.05" y1="41.275" x2="19.05" y2="43.18" width="0.4064" layer="16"/>
+</signal>
+<signal name="N$4">
+<contactref element="J2" pad="3"/>
+<contactref element="U2" pad="13"/>
+<wire x1="16.51" y1="43.18" x2="16.51" y2="41.275" width="0.4064" layer="1"/>
+<wire x1="16.51" y1="41.275" x2="15.24" y2="40.005" width="0.4064" layer="1"/>
+<wire x1="15.24" y1="40.005" x2="13.97" y2="40.005" width="0.4064" layer="1"/>
+<wire x1="13.97" y1="40.005" x2="12.3825" y2="41.5925" width="0.4064" layer="1"/>
+<wire x1="12.3825" y1="41.5925" x2="10.795" y2="41.5925" width="0.4064" layer="1"/>
+<wire x1="10.795" y1="41.5925" x2="10.16" y2="40.9575" width="0.4064" layer="1"/>
+<wire x1="10.16" y1="40.9575" x2="7.3025" y2="38.1" width="0.254" layer="1"/>
+<wire x1="7.3025" y1="38.1" x2="4.605" y2="38.1" width="0.254" layer="1"/>
+</signal>
 </signals>

Commit message: Added values. Added png files.
Parts:
- C7: value (none) -> 100n
- J2: value USB_MICRO_B_2.0-TH -> Micro USB
- R2, R5, R7, R8: value 1k -> 470
- U1: value V_REG_MCP170X -> MCP1702-33
Changed lines of the file:
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@@
 <layer number="21" name="tPlace" color="7" fill="1" visible="yes" active="yes"/>
 <layer number="22" name="bPlace" color="7" fill="1" visible="yes" active="yes"/>
-<layer number="23" name="tOrigins" color="15" fill="1" visible="yes" active="yes"/>
-<layer number="24" name="bOrigins" color="15" fill="1" visible="yes" active="yes"/>
+<layer number="23" name="tOrigins" color="15" fill="1" visible="no" active="yes"/>
+<layer number="24" name="bOrigins" color="15" fill="1" visible="no" active="yes"/>
 <layer number="25" name="tNames" color="7" fill="1" visible="yes" active="yes"/>
 <layer number="26" name="bNames" color="7" fill="1" visible="yes" active="yes"/>
@@
 <layer number="123" name="tTestmark" color="7" fill="1" visible="no" active="yes"/>
 <layer number="124" name="bTestmark" color="7" fill="1" visible="no" active="yes"/>
-<layer number="125" name="_tNames" color="7" fill="1" visible="no" active="yes"/>
+<layer number="125" name="_tNames" color="7" fill="1" visible="yes" active="yes"/>
 <layer number="126" name="_bNames" color="7" fill="1" visible="yes" active="yes"/>
 <layer number="127" name="_tValues" color="7" fill="1" visible="yes" active="yes"/>
 <layer number="128" name="_bValues" color="7" fill="1" visible="yes" active="yes"/>
-<layer number="129" name="Mask" color="7" fill="1" visible="yes" active="yes"/>
+<layer number="129" name="Mask" color="7" fill="1" visible="no" active="yes"/>
 <layer number="131" name="tAdjust" color="7" fill="1" visible="no" active="yes"/>
 <layer number="132" name="bAdjust" color="7" fill="1" visible="no" active="yes"/>
@@
 <attribute name="VALUE" x="43.815" y="11.43" size="0.8128" layer="27" ratio="10" rot="R180"/>
 </element>
-<element name="R8" library="rc-master" package="0207/10" value="1k" x="34.29" y="24.13"/>
+<element name="R8" library="rc-master" package="0207/10" value="470" x="34.29" y="24.13"/>
 <element name="C2" library="rc-master-th" package="C025-040X018" value="100n" x="11.43" y="38.1" smashed="yes" rot="R270">
 <attribute name="NAME" x="10.4775" y="40.9575" size="1.016" layer="25" ratio="18"/>
@@
 <attribute name="NAME" x="39.6875" y="39.37" size="0.8128" layer="26" ratio="18" rot="MR180"/>
 </element>
-<element name="C7" library="rc-master-th" package="C025-040X018" value="" x="45.72" y="37.465" smashed="yes">
+<element name="C7" library="rc-master-th" package="C025-040X018" value="100n" x="45.72" y="37.465" smashed="yes">
 <attribute name="NAME" x="43.4975" y="38.735" size="1.016" layer="25" ratio="18"/>
 <attribute name="VALUE" x="48.895" y="35.8775" size="0.8128" layer="27" ratio="10"/>
@@
 <attribute name="VALUE" x="10.795" y="19.939" size="1.27" layer="27" ratio="10"/>
 </element>
-<element name="R5" library="rc-master" package="0207/7" value="1k" x="16.51" y="19.05" smashed="yes" rot="R180">
+<element name="R5" library="rc-master" package="0207/7" value="470" x="16.51" y="19.05" smashed="yes" rot="R180">
 <attribute name="NAME" x="15.24" y="17.78" size="1.016" layer="25" ratio="18" rot="R180"/>
 <attribute name="VALUE" x="19.05" y="19.685" size="0.8128" layer="27" ratio="10" rot="R180"/>
 </element>
-<element name="R7" library="rc-master" package="0207/7" value="1k" x="16.51" y="22.86" smashed="yes" rot="R180">
+<element name="R7" library="rc-master" package="0207/7" value="470" x="16.51" y="22.86" smashed="yes" rot="R180">
 <attribute name="NAME" x="15.24" y="21.59" size="1.016" layer="25" ratio="18" rot="R180"/>
 <attribute name="VALUE" x="19.05" y="23.495" size="0.8128" layer="27" ratio="10" rot="R180"/>
 </element>
-<element name="U1" library="adi-misc" package="TO-92" value="V_REG_MCP170X" x="24.13" y="12.7" smashed="yes" rot="R90">
+<element name="U1" library="adi-misc" package="TO-92" value="MCP1702-33" x="24.13" y="12.7" smashed="yes" rot="R90">
 <attribute name="NAME" x="26.035" y="12.3825" size="1.016" layer="25" ratio="18"/>
 <attribute name="VALUE" x="25.4" y="15.875" size="0.8128" layer="27" ratio="10" rot="R90"/>
@@
 <attribute name="VALUE" x="10.795" y="30.099" size="1.27" layer="27" ratio="10"/>
 </element>
-<element name="R2" library="rc-master" package="0207/7" value="1k" x="16.51" y="27.94" smashed="yes" rot="R180">
+<element name="R2" library="rc-master" package="0207/7" value="470" x="16.51" y="27.94" smashed="yes" rot="R180">
 <attribute name="NAME" x="15.24" y="26.67" size="1.016" layer="25" ratio="18" rot="R180"/>
 <attribute name="VALUE" x="19.05" y="28.575" size="0.8128" layer="27" ratio="10" rot="R180"/>
@@
 <attribute name="VALUE" x="9.2075" y="53.975" size="0.8128" layer="27" ratio="10" rot="R180"/>
 </element>
-<element name="J2" library="adi-misc" package="ZX62D-AB-5P8" value="USB_MICRO_B_2.0-TH" x="1.905" y="38.1" rot="R270"/>
+<element name="J2" library="adi-misc" package="ZX62D-AB-5P8" value="Micro USB" x="1.905" y="38.1" rot="R270"/>
 </elements>
 <signals>
