File: uino-328th.sch (EAGLE design)
At the start: 38 parts, among them J1 CON_TERMINAL_BLOCK_02-5MM, J2 USB_MICRO_B_2.0-TH, U1 V_REG_MCP170X, U2 PIC16F1454-P, U3 ATMEGA328P-P

Commit message: Some minor final changes.
Connections:
- removed net N$6: J2.ID
Changed lines of the file:
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@@
 <part name="GND17" library="supply1" deviceset="GND" device=""/>
 <part name="GND18" library="supply1" deviceset="GND" device=""/>
-<part name="J2" library="adi-misc" deviceset="USB_MICRO_B_2.0-TH" device=""/>
 <part name="U3" library="adi-atmega" deviceset="ATMEGA328P" device="-P"/>
 <part name="GND16" library="supply1" deviceset="GND" device=""/>
@@
 <part name="S1" library="adi-misc" deviceset="TL1100X" device=""/>
 <part name="GND10" library="supply1" deviceset="GND" device=""/>
+<part name="J2" library="adi-misc" deviceset="USB_MICRO_B_2.0-TH" device=""/>
 </parts>
 <sheets>
@@
 <instance part="GND17" gate="1" x="187.96" y="127"/>
 <instance part="GND18" gate="1" x="187.96" y="48.26"/>
-<instance part="J2" gate="G$1" x="-27.94" y="81.28" rot="MR0"/>
 <instance part="U3" gate="G$1" x="124.46" y="99.06"/>
 <instance part="GND16" gate="1" x="187.96" y="154.94"/>
@@
 <instance part="S1" gate="G$1" x="50.8" y="111.76" rot="R90"/>
 <instance part="GND10" gate="1" x="50.8" y="101.6"/>
+<instance part="J2" gate="G$1" x="-27.94" y="81.28" rot="MR0"/>
 </instances>
 <busses>
@@
 <junction x="-2.54" y="66.04"/>
 <pinref part="J2" gate="G$1" pin="S1"/>
+<wire x1="-27.94" y1="71.12" x2="-27.94" y2="66.04" width="0.1524" layer="91"/>
+<wire x1="-27.94" y1="66.04" x2="-25.4" y2="66.04" width="0.1524" layer="91"/>
+<pinref part="J2" gate="G$1" pin="S2"/>
+<wire x1="-25.4" y1="66.04" x2="-17.78" y2="66.04" width="0.1524" layer="91"/>
+<wire x1="-17.78" y1="66.04" x2="-2.54" y2="66.04" width="0.1524" layer="91"/>
 <wire x1="-25.4" y1="71.12" x2="-25.4" y2="66.04" width="0.1524" layer="91"/>
-<wire x1="-25.4" y1="66.04" x2="-15.24" y2="66.04" width="0.1524" layer="91"/>
+<junction x="-25.4" y="66.04"/>
 <pinref part="J2" gate="G$1" pin="GND"/>
-<wire x1="-15.24" y1="66.04" x2="-2.54" y2="66.04" width="0.1524" layer="91"/>
-<wire x1="-20.32" y1="76.2" x2="-15.24" y2="76.2" width="0.1524" layer="91"/>
-<wire x1="-15.24" y1="76.2" x2="-15.24" y2="66.04" width="0.1524" layer="91"/>
-<junction x="-15.24" y="66.04"/>
-<pinref part="J2" gate="G$1" pin="S2"/>
-<junction x="-25.4" y="71.12"/>
+<wire x1="-20.32" y1="76.2" x2="-17.78" y2="76.2" width="0.1524" layer="91"/>
+<wire x1="-17.78" y1="76.2" x2="-17.78" y2="66.04" width="0.1524" layer="91"/>
+<junction x="-17.78" y="66.04"/>
 </segment>
 <segment>
@@
 <wire x1="154.94" y1="66.04" x2="167.64" y2="66.04" width="0.1524" layer="91"/>
 <label x="167.64" y="66.04" size="1.778" layer="95" rot="MR0"/>
-</segment>
-</net>
-<net name="N$3" class="0">
-<segment>
-<pinref part="J2" gate="G$1" pin="D-"/>
-<pinref part="U2" gate="G$1" pin="RA1(D-)"/>
-<wire x1="-20.32" y1="83.82" x2="0" y2="83.82" width="0.1524" layer="91"/>
-</segment>
-</net>
-<net name="N$4" class="0">
-<segment>
-<pinref part="J2" gate="G$1" pin="D+"/>
-<pinref part="U2" gate="G$1" pin="RA0(D+)"/>
-<wire x1="-20.32" y1="81.28" x2="0" y2="81.28" width="0.1524" layer="91"/>
-</segment>
-</net>
-<net name="N$6" class="0">
-<segment>
-<pinref part="J2" gate="G$1" pin="ID"/>
-<wire x1="-20.32" y1="78.74" x2="-15.24" y2="78.74" width="0.1524" layer="91"/>
 </segment>
 </net>
@@
 <net name="VBUS" class="0">
 <segment>
-<pinref part="J2" gate="G$1" pin="VBUS"/>
-<wire x1="-20.32" y1="86.36" x2="-7.62" y2="86.36" width="0.1524" layer="91"/>
-<label x="-7.62" y="86.36" size="1.778" layer="95" rot="MR0"/>
-</segment>
-<segment>
 <pinref part="F1" gate="G$1" pin="1"/>
 <wire x1="-25.4" y1="167.64" x2="-33.02" y2="167.64" width="0.1524" layer="91"/>
 <label x="-33.02" y="167.64" size="1.778" layer="95"/>
 </segment>
+<segment>
+<pinref part="J2" gate="G$1" pin="VBUS"/>
+<wire x1="-20.32" y1="86.36" x2="-10.16" y2="86.36" width="0.1524" layer="91"/>
+<label x="-10.16" y="86.36" size="1.778" layer="95" rot="MR0"/>
+</segment>
 </net>
 <net name="N$14" class="0">
@@
 </segment>
 </net>
+<net name="N$3" class="0">
+<segment>
+<pinref part="J2" gate="G$1" pin="D-"/>
+<pinref part="U2" gate="G$1" pin="RA1(D-)"/>
+<wire x1="-20.32" y1="83.82" x2="0" y2="83.82" width="0.1524" layer="91"/>
+</segment>
+</net>
+<net name="N$4" class="0">
+<segment>
+<pinref part="J2" gate="G$1" pin="D+"/>
+<pinref part="U2" gate="G$1" pin="RA0(D+)"/>
+<wire x1="-20.32" y1="81.28" x2="0" y2="81.28" width="0.1524" layer="91"/>
+</segment>
+</net>

Commit message: Added values. Added png files.
Parts:
- C7: value (none) -> 100n
- J2: value USB_MICRO_B_2.0-TH -> Micro USB
- R2, R5, R7, R8: value 1k -> 470
- U1: value V_REG_MCP170X -> MCP1702-33
Changed lines of the file:
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@@
 <layer number="91" name="Nets" color="2" fill="1" visible="yes" active="yes"/>
 <layer number="92" name="Busses" color="1" fill="1" visible="yes" active="yes"/>
-<layer number="93" name="Pins" color="2" fill="1" visible="yes" active="yes"/>
+<layer number="93" name="Pins" color="2" fill="1" visible="no" active="yes"/>
 <layer number="94" name="Symbols" color="4" fill="1" visible="yes" active="yes"/>
 <layer number="95" name="Names" color="7" fill="1" visible="yes" active="yes"/>
@@
 <part name="C8" library="rc-master-th" deviceset="C_" device="C025-040X018" value="100n"/>
 <part name="GND12" library="supply1" deviceset="GND" device=""/>
-<part name="R8" library="rc-master" deviceset="R_" device="X0207/10" value="1k"/>
+<part name="R8" library="rc-master" deviceset="R_" device="X0207/10" value="470"/>
 <part name="SUPPLY3" library="SparkFun-Aesthetics" deviceset="VCC" device=""/>
 <part name="GND4" library="supply1" deviceset="GND" device=""/>
@@
 <part name="JP2" library="jumpers" deviceset="SJ-" device="035"/>
 <part name="JP1" library="jumpers" deviceset="SJ-" device="035"/>
-<part name="C7" library="rc-master-th" deviceset="C_" device="C025-040X018"/>
+<part name="C7" library="rc-master-th" deviceset="C_" device="C025-040X018" value="100n"/>
 <part name="SUPPLY6" library="SparkFun-Aesthetics" deviceset="VCC" device=""/>
 <part name="SUPPLY1" library="SparkFun-Aesthetics" deviceset="VCC" device=""/>
@@
 <part name="D5" library="SparkFun-LED" deviceset="LED" device="3MM" value="Yellow"/>
 <part name="D4" library="SparkFun-LED" deviceset="LED" device="3MM" value="Yellow"/>
-<part name="R5" library="rc-master" deviceset="R_" device="X0207/7" value="1k"/>
-<part name="R7" library="rc-master" deviceset="R_" device="X0207/7" value="1k"/>
+<part name="R5" library="rc-master" deviceset="R_" device="X0207/7" value="470"/>
+<part name="R7" library="rc-master" deviceset="R_" device="X0207/7" value="470"/>
 <part name="SUPPLY9" library="SparkFun-Aesthetics" deviceset="VCC" device=""/>
 <part name="SUPPLY7" library="SparkFun-Aesthetics" deviceset="VCC" device=""/>
-<part name="U1" library="adi-misc" deviceset="V_REG_MCP170X" device=""/>
+<part name="U1" library="adi-misc" deviceset="V_REG_MCP170X" device="" value="MCP1702-33"/>
 <part name="J1" library="adi-misc" deviceset="CON_TERMINAL_BLOCK_02" device="-5MM"/>
 <part name="D1" library="diode" deviceset="SCHOTTKY-DIODE" device="DO35-7"/>
@@
 <part name="SUPPLY2" library="SparkFun-Aesthetics" deviceset="VIN" device=""/>
 <part name="D3" library="SparkFun-LED" deviceset="LED" device="3MM" value="Green"/>
-<part name="R2" library="rc-master" deviceset="R_" device="X0207/7" value="1k"/>
+<part name="R2" library="rc-master" deviceset="R_" device="X0207/7" value="470"/>
 <part name="SUPPLY5" library="SparkFun-Aesthetics" deviceset="VCC" device=""/>
 <part name="GND11" library="supply1" deviceset="GND" device=""/>
@@
 <part name="S1" library="adi-misc" deviceset="TL1100X" device=""/>
 <part name="GND10" library="supply1" deviceset="GND" device=""/>
-<part name="J2" library="adi-misc" deviceset="USB_MICRO_B_2.0-TH" device=""/>
+<part name="J2" library="adi-misc" deviceset="USB_MICRO_B_2.0-TH" device="" value="Micro USB"/>
 </parts>
 <sheets>
@@
 <instance part="SUPPLY9" gate="G$1" x="93.98" y="170.18"/>
 <instance part="SUPPLY7" gate="G$1" x="76.2" y="170.18"/>
-<instance part="U1" gate="G$1" x="7.62" y="157.48"/>
+<instance part="U1" gate="G$1" x="7.62" y="157.48" smashed="yes">
+<attribute name="NAME" x="10.16" y="149.86" size="1.778" layer="95"/>
+<attribute name="VALUE" x="-0.762" y="161.29" size="1.778" layer="96"/>
+</instance>
 <instance part="J1" gate="CON" x="-30.48" y="154.94" rot="R180"/>
 <instance part="D1" gate="G$1" x="-12.7" y="149.86" rot="R90"/>
@@
 <instance part="S1" gate="G$1" x="50.8" y="111.76" rot="R90"/>
 <instance part="GND10" gate="1" x="50.8" y="101.6"/>
-<instance part="J2" gate="G$1" x="-27.94" y="81.28" rot="MR0"/>
+<instance part="J2" gate="G$1" x="-27.94" y="81.28" smashed="yes" rot="MR0">
+<attribute name="NAME" x="-22.86" y="95.25" size="1.778" layer="95" rot="MR0"/>
+<attribute name="VALUE" x="-22.86" y="91.44" size="1.778" layer="96" rot="MR0"/>
+</instance>
 </instances>
 <busses>
